Commit message: Adjust torque limit in URDF

File: resources/anymal_c/urdf/anymal_with_anklepitch_sim.urdf (robot description, URDF)
Before this commit: robot anymal, 86 links, 85 joints
Joints:
- joint LH_ANKLE_pitch: limit lower=-0.78539816339 upper=0.78539816339 effort=180.0 velocity=10.0 -> lower=-0.78539816339 upper=0.78539816339 effort=80.0 velocity=10.0
- joint RH_ANKLE_pitch: limit lower=-0.78539816339 upper=0.78539816339 effort=180.0 velocity=10.0 -> lower=-0.78539816339 upper=0.78539816339 effort=80.0 velocity=10.0
